File: KicadEuropower/KicadEuropower.kicad_pcb (KiCad board)
At the start: 2 copper layers, 100 x 100 mm, 19 parts, among them P1 Doepfer_Power_10pin, P10 Doepfer_Power_10pin, P11 Doepfer_Power_10pin, P12 Doepfer_Power_10pin, P13 Doepfer_Power_10pin, P14 Doepfer_Power_10pin, P2 Doepfer_Power_16pin, P3 Doepfer_Power_10pin, P4 Doepfer_Power_16pin, P5 Doepfer_Power_10pin, P6 Doepfer_Power_16pin, P7 Doepfer_Power_10pin, P8 Doepfer_Power_16pin, P9 Doepfer_Power_10pin, T1 Transformer_1P_2S

Commit message: PCB Placement started
Parts:
- removed T1: Transformer_1P_2S, Transformers_SMPS_ThroughHole:ETD29_13Pin_Horizontal_EPCOS-B66359A1013T
- added C1: 100n, Capacitor_SMD:C_0805_2012Metric_Pad1.15x1.40mm_HandSolder, B.Cu at (109.2, 135.7)
- added C10: 1000uF, Capacitor_THT:CP_Radial_D8.0mm_P3.80mm, F.Cu at (20.8, -11.3)
- added C11: 1000uF, Capacitor_THT:CP_Radial_D8.0mm_P3.80mm, F.Cu at (37.7, -21.6)
- added C12: 1000uF, Capacitor_THT:CP_Radial_D8.0mm_P3.80mm, F.Cu at (48.5, 94.0)
- added C13: 100n, Capacitor_SMD:C_0805_2012Metric_Pad1.15x1.40mm_HandSolder, B.Cu at (42.4, 112.2)
- added C14: 100n, Capacitor_SMD:C_0805_2012Metric_Pad1.15x1.40mm_HandSolder, B.Cu at (23.1, 120.6)
- added C15: 100n, Capacitor_SMD:C_0805_2012Metric_Pad1.15x1.40mm_HandSolder, B.Cu at (45.9, 120.2)
- added C16: 100n, Capacitor_SMD:C_0805_2012Metric_Pad1.15x1.40mm_HandSolder, B.Cu at (105.5, 135.7)
- added C17: 100n, Capacitor_SMD:C_0805_2012Metric_Pad1.15x1.40mm_HandSolder, B.Cu at (101.7, 135.7)
- added C18: 100n, Capacitor_SMD:C_0805_2012Metric_Pad1.15x1.40mm_HandSolder, B.Cu at (29.9, 110.6)
- added C19: 100n, Capacitor_SMD:C_0805_2012Metric_Pad1.15x1.40mm_HandSolder, B.Cu at (34.9, 112.2)
- added C2: 100n, Capacitor_SMD:C_0805_2012Metric_Pad1.15x1.40mm_HandSolder, B.Cu at (53.4, 126.1)
- added C20: 100n, Capacitor_SMD:C_0805_2012Metric_Pad1.15x1.40mm_HandSolder, B.Cu at (26.1, 110.6)
- added C21: 100n, Capacitor_SMD:C_0805_2012Metric_Pad1.15x1.40mm_HandSolder, B.Cu at (109.0, 133.7)
- added C22: 100n, Capacitor_SMD:C_0805_2012Metric_Pad1.15x1.40mm_HandSolder, B.Cu at (22.4, 110.6)
- added C23: 100n, Capacitor_SMD:C_0805_2012Metric_Pad1.15x1.40mm_HandSolder, B.Cu at (114.2, 117.7)
- added C24: 100n, Capacitor_SMD:C_0805_2012Metric_Pad1.15x1.40mm_HandSolder, B.Cu at (23.1, 118.7)
- added C25: 100n, Capacitor_SMD:C_0805_2012Metric_Pad1.15x1.40mm_HandSolder, B.Cu at (32.2, 121.2)
- added C26: 100n, Capacitor_SMD:C_0805_2012Metric_Pad1.15x1.40mm_HandSolder, B.Cu at (32.2, 119.2)
- added C27: 100n, Capacitor_SMD:C_0805_2012Metric_Pad1.15x1.40mm_HandSolder, B.Cu at (114.2, 115.7)
- added C28: 100n, Capacitor_SMD:C_0805_2012Metric_Pad1.15x1.40mm_HandSolder, B.Cu at (38.7, 112.2)
- added C29: 100n, Capacitor_SMD:C_0805_2012Metric_Pad1.15x1.40mm_HandSolder, B.Cu at (56.6, 111.5)
- added C3: 1000uF, Capacitor_THT:CP_Radial_D8.0mm_P3.80mm, F.Cu at (39.3, -13.0)
- added C30: 100n, Capacitor_SMD:C_0805_2012Metric_Pad1.15x1.40mm_HandSolder, B.Cu at (118.0, 115.7)
- added C31: 100n, Capacitor_SMD:C_0805_2012Metric_Pad1.15x1.40mm_HandSolder, B.Cu at (45.9, 126.1)
- added C32: 100n, Capacitor_SMD:C_0805_2012Metric_Pad1.15x1.40mm_HandSolder, B.Cu at (45.9, 124.1)
- added C33: 100n, Capacitor_SMD:C_0805_2012Metric_Pad1.15x1.40mm_HandSolder, B.Cu at (52.8, 111.5)
- added C34: 100n, Capacitor_SMD:C_0805_2012Metric_Pad1.15x1.40mm_HandSolder, B.Cu at (34.1, 106.9)
- added C35: 100n, Capacitor_SMD:C_0805_2012Metric_Pad1.15x1.40mm_HandSolder, B.Cu at (108.3, 144.6)
- added C36: 100n, Capacitor_SMD:C_0805_2012Metric_Pad1.15x1.40mm_HandSolder, B.Cu at (49.7, 126.1)
- added C37: 100n, Capacitor_SMD:C_0805_2012Metric_Pad1.15x1.40mm_HandSolder, B.Cu at (52.8, 109.6)
- added C38: 100n, Capacitor_SMD:C_0805_2012Metric_Pad1.15x1.40mm_HandSolder, B.Cu at (118.0, 117.7)
- added C39: 100n, Capacitor_SMD:C_0805_2012Metric_Pad1.15x1.40mm_HandSolder, B.Cu at (49.7, 124.1)
- added C4: 1000uF, Capacitor_THT:CP_Radial_D8.0mm_P3.80mm, F.Cu at (111.4, 68.8)
- added C40: 100n, Capacitor_SMD:C_0805_2012Metric_Pad1.15x1.40mm_HandSolder, B.Cu at (52.8, 107.6)
- added C41: 100n, Capacitor_SMD:C_0805_2012Metric_Pad1.15x1.40mm_HandSolder, B.Cu at (108.3, 142.7)
- added C42: 100n, Capacitor_SMD:C_0805_2012Metric_Pad1.15x1.40mm_HandSolder, B.Cu at (37.8, 106.9)
- added C5: 1000uF, Capacitor_THT:CP_Radial_D8.0mm_P3.80mm, F.Cu at (19.0, 94.0)
- added C6: 1000uF, Capacitor_THT:CP_Radial_D8.0mm_P3.80mm, F.Cu at (51.6, -30.2)
- added C7: 1000uF, Capacitor_THT:CP_Radial_D8.0mm_P3.80mm, F.Cu at (78.0, 94.0)
- added C8: 100n, Capacitor_SMD:C_0805_2012Metric_Pad1.15x1.40mm_HandSolder, B.Cu at (45.9, 122.2)
- added C9: 1000uF, Capacitor_THT:CP_Radial_D8.0mm_P3.80mm, F.Cu at (108.4, 60.2)
- added D1: 1N4001, Diode_THT:D_DO-41_SOD81_P10.16mm_Horizontal, F.Cu at (33.9, 37.2)
- added D2: 1N4001, Diode_THT:D_DO-41_SOD81_P10.16mm_Horizontal, F.Cu at (54.0, 24.0)
- added D3: LED, LED_SMD:LED_0805_2012Metric_Pad1.15x1.40mm_HandSolder, F.Cu at (62.0, 14.0)
- added D4: LED, LED_SMD:LED_0805_2012Metric_Pad1.15x1.40mm_HandSolder, F.Cu at (12.9, 31.2)
- added D5: LED, LED_SMD:LED_0805_2012Metric_Pad1.15x1.40mm_HandSolder, F.Cu at (14.0, 9.00)
- added D6: 1N4001, Diode_THT:D_DO-41_SOD81_P10.16mm_Horizontal, F.Cu at (13.0, 19.0)
- added D7: LED, LED_SMD:LED_0805_2012Metric_Pad1.15x1.40mm_HandSolder, F.Cu at (85.0, 27.0)
- added D8: LED, LED_SMD:LED_0805_2012Metric_Pad1.15x1.40mm_HandSolder, F.Cu at (85.0, 17.0)
- added D9: LED, LED_SMD:LED_0805_2012Metric_Pad1.15x1.40mm_HandSolder, F.Cu at (85.0, 9.00)
- added FL1: EMI_Filter_CommonMode, Choke_Toroid_ThroughHole:Transformer_Toroid_horizontal_Diameter9mm_Amidon-T30, F.Cu at (42.0, 13.0)
- added FL2: EMI_Filter_CommonMode, Choke_Toroid_ThroughHole:Transformer_Toroid_horizontal_Diameter9mm_Amidon-T30, F.Cu at (80.0, 13.0)
- added FL3: EMI_Filter_CommonMode, Choke_Toroid_ThroughHole:Transformer_Toroid_horizontal_Diameter9mm_Amidon-T30, F.Cu at (30.0, 13.0)
- added J1: Conn_01x02_Male, TerminalBlock:TerminalBlock_Altech_AK300-2_P5.00mm, F.Cu at (59.0, 6.00)
- added J2: Conn_01x02_Male, TerminalBlock:TerminalBlock_Altech_AK300-2_P5.00mm, F.Cu at (72.0, 6.00)
- added J3: Conn_01x02_Male, TerminalBlock:TerminalBlock_Altech_AK300-2_P5.00mm, F.Cu at (94.0, 9.00)
- added J4: Conn_01x03_Male, TerminalBlock:TerminalBlock_Altech_AK300-3_P5.00mm, F.Cu at (5.00, 4.00)
- added J5: Conn_01x03_Male, TerminalBlock:TerminalBlock_Altech_AK300-3_P5.00mm, F.Cu at (4.92, 26.2)
- added J6: Conn_01x03_Male, TerminalBlock:TerminalBlock_Altech_AK300-3_P5.00mm, F.Cu at (94.0, 27.0)
- added R1: 680R, Resistor_SMD:R_0805_2012Metric_Pad1.15x1.40mm_HandSolder, B.Cu at (73.0, 32.5)
- added R2: 3k3, Resistor_SMD:R_0805_2012Metric_Pad1.15x1.40mm_HandSolder, B.Cu at (68.8, 32.1)
- added R3: 3k3, Resistor_SMD:R_0805_2012Metric_Pad1.15x1.40mm_HandSolder, B.Cu at (73.0, 30.6)
- added R4: 1k5, Resistor_SMD:R_0805_2012Metric_Pad1.15x1.40mm_HandSolder, B.Cu at (73.0, 28.6)
- added R5: 1k5, Resistor_SMD:R_0805_2012Metric_Pad1.15x1.40mm_HandSolder, B.Cu at (67.2, 35.7)
- added R6: 680R, Resistor_SMD:R_0805_2012Metric_Pad1.15x1.40mm_HandSolder, B.Cu at (73.0, 26.4)
- added RV1: Varistor, Varistor:RV_Disc_D12mm_W4.8mm_P7.5mm, F.Cu at (21.9, 26.2)
- added RV3: Varistor, Varistor:RV_Disc_D12mm_W4.8mm_P7.5mm, F.Cu at (28.9, 38.2)
- added U1: LM7812_TO220, Package_TO_SOT_THT:TO-220-3_Vertical, F.Cu at (40.0, 3.00)
- added U2: LM7805_TO220, Package_TO_SOT_THT:TO-220-3_Vertical, F.Cu at (79.0, 3.00)
- added U3: LM7912_TO220, Package_TO_SOT_THT:TO-220-3_Vertical, F.Cu at (29.0, 3.00)
- F1, F3: moved to B.Cu
- moved RV2 149.6 mm to (71.2, 23.0), turned to 90 degrees
- moved F2 142.4 mm to (54.0, 17.0)
- moved F1 119.9 mm to (14.7, 26.4)
- moved F3 114.1 mm to (14.7, 36.2)
- renumbered RV1 to RV2
Connections:
- F1 pad 1: (no net) -> /+15v-ext
- F1 pad 2: (no net) -> Net-(D1-Pad2)
- F2 pad 1: Net-(F2-Pad1) -> /+5V-ext
- F3 pad 1: (no net) -> /-15v-ext
- F3 pad 2: (no net) -> Net-(D6-Pad1)
- P1 pad 3: (no net) -> GND
- P1 pad 7: (no net) -> GND
- P5 pad 3: (no net) -> GND
- P5 pad 7: (no net) -> GND
- P7 pad 3: (no net) -> GND
- P7 pad 7: (no net) -> GND
Other:
- net class Default: clearance 0.2 -> 0.25; trace_width 0.25 -> 0.75; via_dia 0.8 -> 1; via_drill 0.4 -> 0.5
- net class Power added: clearance 0.25, trace_width 1, via_dia 1.2, via_drill 0.7
- rule trace_clearance: 0.2 -> 0.25

Commit message: 3D shapes init
Parts:
- moved C4 84.3 mm to (52.0, 9.00)
- moved C9 52.1 mm to (64.0, 33.0)
- moved C3 48.1 mm to (28.7, 33.9), turned to 270 degrees
- moved C10 45.2 mm to (19.7, 33.9), turned to 270 degrees
- moved C6 41.1 mm to (64.0, 9.00)
- moved R1 39.3 mm to (112.0, 27.5)
- moved R2 39.3 mm to (107.8, 27.1)
- moved R3 39.3 mm to (112.0, 25.6)
- moved R6 39.3 mm to (112.0, 21.4)
- moved R4 39.2 mm to (112.0, 24.3)
- moved R5 39.0 mm to (106.2, 34.3)
- moved C21 38.3 mm to (77.0, 112.7)
- moved C35 38.3 mm to (76.3, 123.6)
- moved C1 38.3 mm to (77.2, 114.7)
- moved C16 38.3 mm to (73.5, 114.7)
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