File: KicadEuropower/KicadEuropower.kicad_pcb (KiCad board)
At the start: 2 copper layers, 100 x 100 mm, 89 parts, among them J1 Conn_01x02_Male, J2 Conn_01x02_Male, J3 Conn_01x02_Male, J4 Conn_01x03_Male, J5 Conn_01x03_Male, J6 Conn_01x03_Male, P1 Doepfer_Power_10pin, P10 Doepfer_Power_10pin, P11 Doepfer_Power_10pin, P12 Doepfer_Power_10pin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

Commit message: Component placement update
Parts:
- removed P13, P14: Doepfer_Power_10pin, Connectors_IDC:IDC-Header_2x05_Pitch2.54mm_Straight
- added C43: 100n, Capacitor_SMD:C_0805_2012Metric_Pad1.15x1.40mm_HandSolder, F.Cu at (66.6, 105.1)
- added C44: 100n, Capacitor_SMD:C_0805_2012Metric_Pad1.15x1.40mm_HandSolder, F.Cu at (66.6, 107.1)
- C10, C11, C3, C5, C6: footprint Capacitor_THT:CP_Radial_D8.0mm_P3.80mm -> Capacitor_THT:CP_Radial_D10.0mm_P5.00mm
- C13, C14, C8: value 100n -> 1000uF; footprint Capacitor_SMD:C_0805_2012Metric_Pad1.15x1.40mm_HandSolder -> Capacitor_THT:CP_Radial_D10.0mm_P5.00mm; moved to F.Cu
- C9: value 1000uF -> 100n; footprint Capacitor_THT:CP_Radial_D8.0mm_P3.80mm -> Capacitor_SMD:C_0805_2012Metric_Pad1.15x1.40mm_HandSolder; moved to B.Cu
- moved C7 86.3 mm to (63.5, 8.89)
- moved C12 85.5 mm to (40.2, 8.89)
- moved C6 74.3 mm to (48.3, 81.6)
- moved C13 64.2 mm to (48.3, 48.3)
- moved C14 56.1 mm to (48.3, 70.5)
- moved C5 45.3 mm to (48.3, 59.4)
- moved C10 43.2 mm to (62.9, 33.0), turned to 0 degrees
- moved C9 34.8 mm to (86.4, 6.35)
- moved C8 29.5 mm to (48.3, 92.7)
- moved C11 24.0 mm to (39.4, 33.0)
- moved C3 22.4 mm to (51.2, 33.0), turned to 0 degrees
- moved P12 14.7 mm to (34.3, 48.5)
- moved D1 4.50 mm to (34.0, 26.0)
- moved D6 3.97 mm to (16.0, 16.0)
- moved RV1 3.72 mm to (28.0, 16.7)
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Connections:
- net /+15v-ext renamed Vin+15
- net /-15v-ext renamed Vin-15
- net Net-(C1-Pad1) renamed /+15v-int
- C11 pad 1: GND -> VinGND
- C12 pad 2: -12V -> /-15v-int
- C13 pad 2: Net-(C11-Pad2) -> -12V
- C14 pad 1: -12V -> GND
- C14 pad 2: GND -> -12V
- C15 pad 1: -12V -> GND
- C15 pad 2: GND -> /-15v-int
- C26 pad 1: GND -> -12V
- C26 pad 2: +12V -> GND
- C27 pad 1: GND -> -12V
- C27 pad 2: +12V -> GND
- C3 pad 2: Net-(C10-Pad1) -> VinGND
- C38 pad 1: +5V -> GND
- C38 pad 2: GND -> +12V
- C39 pad 1: +5V -> GND
- C39 pad 2: GND -> +12V
- C6 pad 1: Net-(C2-Pad1) -> +12V
- C7 pad 1: +5V -> Net-(C2-Pad1)
- C8 pad 1: /+5V-ext -> +5V
- C8 pad 2: Net-(C8-Pad2) -> GND
- C9 pad 1: Net-(C9-Pad1) -> /+5V-ext
- C9 pad 2: Net-(C8-Pad2) -> Net-(C10-Pad2)
- D2 pad 1: Net-(C9-Pad1) -> Net-(C10-Pad1)
- D3 pad 1: Net-(C8-Pad2) -> Net-(C10-Pad2)
- D6 pad 2: Net-(C10-Pad2) -> Net-(C11-Pad2)
- FL1 pad 1: Net-(C10-Pad1) -> VinGND
- FL2 pad 1: Net-(C8-Pad2) -> Net-(C10-Pad2)
- FL2 pad 3: Net-(C9-Pad1) -> Net-(C10-Pad1)
- FL3 pad 1: Net-(C10-Pad2) -> Net-(C11-Pad2)
- FL3 pad 2: Net-(C11-Pad2) -> /-15v-int
- FL3 pad 3: Net-(C10-Pad1) -> VinGND
- J1 pad 2: Net-(C8-Pad2) -> Net-(C10-Pad2)
- J2 pad 2: Net-(C8-Pad2) -> Net-(C10-Pad2)
- J4 pad 2: Net-(C10-Pad1) -> VinGND
- J5 pad 2: Net-(C10-Pad1) -> VinGND
- RV1 pad 2: Net-(C10-Pad1) -> VinGND
- RV2 pad 2: Net-(C8-Pad2) -> Net-(C10-Pad2)
- RV3 pad 1: Net-(C10-Pad1) -> VinGND
- U3 pad 2: Net-(C11-Pad2) -> /-15v-int

Commit message: Mounting holes and Text
Parts:
- added Q1: BD139, Package_TO_SOT_THT:TO-126-3_Vertical, F.Cu at (2.54, 27.9)
- added Q2: BD140, Package_TO_SOT_THT:TO-126-3_Vertical, F.Cu at (2.54, 38.1)
- added R10: 330r, Resistor_SMD:R_0805_2012Metric_Pad1.15x1.40mm_HandSolder, B.Cu at (16.8, 36.8)
- added R11: 10r, Resistor_THT:R_Axial_DIN0204_L3.6mm_D1.6mm_P2.54mm_Vertical, F.Cu at (5.08, 38.1)
- added R7: 10r, Resistor_THT:R_Axial_DIN0204_L3.6mm_D1.6mm_P2.54mm_Vertical, F.Cu at (5.08, 25.4)
- added R8: 330r, Resistor_SMD:R_0805_2012Metric_Pad1.15x1.40mm_HandSolder, B.Cu at (13.7, 34.3)
- added R9: 330r, Resistor_SMD:R_0805_2012Metric_Pad1.15x1.40mm_HandSolder, B.Cu at (6.00, 30.5)
- added REF**: MountingHole_3.2mm_M3_Pad_Via, MountingHole:MountingHole_3.2mm_M3_Pad_Via, F.Cu at (84.0, 16.0)
- added REF**: MountingHole_3.2mm_M3_Pad_Via, MountingHole:MountingHole_3.2mm_M3_Pad_Via, F.Cu at (4.00, 16.0)
- added REF**: MountingHole_3.2mm_M3_Pad_Via, MountingHole:MountingHole_3.2mm_M3_Pad_Via, F.Cu at (96.0, 96.2)
- added REF**: MountingHole_3.2mm_M3_Pad_Via, MountingHole:MountingHole_3.2mm_M3_Pad_Via, F.Cu at (3.75, 96.2)
- added U4: TL071, Package_DIP:DIP-8_W7.62mm_Socket, F.Cu at (10.2, 39.4)
- moved R3 100.1 mm to (13.0, 10.5), turned to 180 degrees
- moved R2 80.0 mm to (29.5, 10.5), turned to 180 degrees
- moved R1 29.8 mm to (95.0, 3.00)
- moved R4 26.9 mm to (89.5, 39.0), turned to 180 degrees
- moved R6 22.6 mm to (89.5, 19.0), turned to 270 degrees
- moved D2 19.0 mm to (73.3, 41.1), turned to 90 degrees
- moved R5 16.7 mm to (89.5, 34.0), turned to 180 degrees
- moved P5 14.7 mm to (93.0, 71.0)
- moved P8 14.7 mm to (78.3, 71.0)
- moved P11 14.7 mm to (5.00, 71.0)
- moved P4 14.7 mm to (19.7, 71.0)
- moved D3 11.8 mm to (98.0, 2.00)
- moved F2 5.10 mm to (79.0, 16.0), turned to 270 degrees
- moved RV2 4.75 mm to (79.3, 32.1), turned to 270 degrees
- moved J2 3.00 mm to (93.0, 6.00)
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Other:
- board text added: "+"
- board text added: "+15V thru"
- board text added: "+15Vin"
- board text added: "-"
- board text added: "-15"
- board text added: "-15V"
- board text added: "5V out"
- board text added: "7V in"
- board text added: "7V thru"
- board text added: "GND"
- board text added: "Reg Out"
- board text added: "V-GND"
- board text added: "in"

Commit message: Groundplanes placed
Parts:
- added C45: 220n, Capacitor_SMD:C_0805_2012Metric_Pad1.15x1.40mm_HandSolder, B.Cu at (13.0, 36.8)
- added C46: 220n, Capacitor_SMD:C_0805_2012Metric_Pad1.15x1.40mm_HandSolder, B.Cu at (8.97, 35.5)
- added JP1: Jumper_2_Open, Connector_PinSocket_2.54mm:PinSocket_1x02_P2.54mm_Vertical, F.Cu at (52.0, 5.50)
- added JP2: Jumper_2_Open, Connector_PinSocket_2.54mm:PinSocket_1x02_P2.54mm_Vertical, F.Cu at (41.0, 5.50)
- added TP1: TestPoint, Connector_PinSocket_2.54mm:PinSocket_1x01_P2.54mm_Vertical, F.Cu at (34.0, 29.0)
- added TP2: Vin+15, Connector_PinSocket_2.54mm:PinSocket_1x01_P2.54mm_Vertical, F.Cu at (6.00, 28.0)
- added TP3: VGnd, Connector_PinSocket_2.54mm:PinSocket_1x01_P2.54mm_Vertical, F.Cu at (6.00, 33.0)
- added TP4: Vin-15, Connector_PinSocket_2.54mm:PinSocket_1x01_P2.54mm_Vertical, F.Cu at (6.00, 36.5)
- C43, C44: moved to B.Cu
- moved C2 110.2 mm to (65.5, 16.5)
- moved C15 103.8 mm to (41.0, 16.5)
- moved C1 101.0 mm to (53.5, 16.5)
- moved C44 100.6 mm to (69.5, 6.50), turned to 270 degrees
- moved C20 88.7 mm to (90.4, 49.5), turned to 270 degrees
- moved C30 82.7 mm to (10.4, 80.0), turned to 270 degrees
- moved C18 76.5 mm to (75.9, 49.5), turned to 270 degrees
- moved C25 74.7 mm to (10.2, 49.8), turned to 270 degrees
- moved C32 73.2 mm to (75.9, 57.4), turned to 270 degrees
- moved C29 71.1 mm to (10.2, 57.7), turned to 270 degrees
- moved C31 70.3 mm to (61.2, 57.4), turned to 270 degrees
- moved C26 69.8 mm to (24.9, 49.8), turned to 270 degrees
- moved C19 67.9 mm to (61.2, 49.5), turned to 270 degrees
- moved C16 64.6 mm to (24.9, 72.1), turned to 270 degrees
- moved C22 63.4 mm to (39.4, 49.5), turned to 270 degrees
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Connections:
- net Net-(C10-Pad2) renamed GNDPWR
Routing:
- added copper zone on F.Cu, net GND
- added copper zone on F.Cu, net GNDPWR
- added copper zone on F.Cu, net VinGND
Other:
- outline, holes or cut-outs redrawn
- board text added: "Bypass +reg"
- board text added: "Bypass -reg"
- board text added: "EURORACK PWR"
- board text added: "Johansen Engineering"
- board text added: "Rev A - 2019/02"
