File: KicadEuropower/_saved_KicadEuropower.sch (KiCad schematic (older format))
At the start: 89 parts, among them J1 Conn_01x02_Male, J2 Conn_01x02_Male, J3 Conn_01x02_Male, J4 Conn_01x03_Male, J5 Conn_01x03_Male, J6 Conn_01x03_Male, P1 Doepfer_Power_10pin, P10 Doepfer_Power_10pin, P11 Doepfer_Power_10pin, P12 Doepfer_Power_10pin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

Commit message: 3D shapes init
Parts:
- removed P13, P14: Doepfer_Power_10pin, Connectors_IDC:IDC-Header_2x05_Pitch2.54mm_Straight, symbol Eurorack:Doepfer_Power_10pin
- U3: value LM7812_TO220 -> LM7912_TO220; symbol Regulator_Linear:LM7812_TO220 -> Regulator_Linear:LM7912_TO220
Connections:
- net labels added: +15v-int, -15v-int, Vin+15, Vin-15, VinGND
- net labels removed: +15v-ext, -15v-ext
- wire segments 525 -> 486
