File: KicadEuropower/_saved_KicadEuropower.sch (KiCad schematic (older format))
At the start: 105 parts, among them J1 Conn_01x02_Male, J2 Conn_01x02_Male, J3 Conn_01x02_Male, J4 Conn_01x03_Male, J5 Conn_01x03_Male, J6 Conn_01x03_Male, P1 Doepfer_Power_10pin, P10 Doepfer_Power_10pin, P11 Doepfer_Power_10pin, P12 Doepfer_Power_10pin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

Commit message: Rev A - Mechanical + Component placement + Text
Parts:
- TP1: value TestPoint -> VGnd
Changed lines of the file:
@@
 P 8400 1350
 F 0 "TP1" H 8458 1470 50  0000 L CNN
-F 1 "TestPoint" H 8458 1379 50  0000 L CNN
+F 1 "VGnd" H 8458 1379 50  0000 L CNN
 F 2 "Connector_PinSocket_2.54mm:PinSocket_1x01_P2.54mm_Vertical" H 8600 1350 50  0001 C CNN
 F 3 "~" H 8600 1350 50  0001 C CNN
