File: KicadEuropower/_autosave-KicadEuropower.kicad_pcb (KiCad board)
At the start: 2 copper layers, 100 x 100 mm, 89 parts, among them J1 Conn_01x02_Male, J2 Conn_01x02_Male, J3 Conn_01x02_Male, J4 Conn_01x03_Male, J5 Conn_01x03_Male, J6 Conn_01x03_Male, P1 Doepfer_Power_10pin, P10 Doepfer_Power_10pin, P11 Doepfer_Power_10pin, P12 Doepfer_Power_10pin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

Commit message: Footprint updates
Parts:
- C10, C3: footprint Capacitor_THT:CP_Radial_D8.0mm_P3.80mm -> Capacitor_THT:CP_Radial_D10.0mm_P5.00mm
- moved C3 23.3 mm to (52.0, 33.0), turned to 0 degrees
- moved C10 20.3 mm to (40.0, 33.0), turned to 0 degrees
- moved D1 4.50 mm to (34.0, 26.0)
- moved D6 3.97 mm to (16.0, 16.0)
- moved RV1 3.72 mm to (28.0, 16.7)
- moved RV3 3.70 mm to (20.7, 24.2)
- moved F3 0.95 mm to (19.6, 15.6)
- moved F1 0.83 mm to (31.2, 15.6)
Connections:
- net /+15v-ext renamed Vin+15
- net /-15v-ext renamed Vin-15
- net Net-(C1-Pad1) renamed /+15v-int
- net Net-(C10-Pad1) renamed VinGND
- net Net-(C11-Pad2) renamed /-15v-int
