File: KicadEuropower/KicadEuropower.sch (KiCad schematic (older format))
At the start: 24 parts, among them P1 Doepfer_Power_10pin, P10 Doepfer_Power_10pin, P11 Doepfer_Power_10pin, P12 Doepfer_Power_10pin, P13 Doepfer_Power_10pin, P14 Doepfer_Power_10pin, P2 Doepfer_Power_16pin, P3 Doepfer_Power_10pin, P4 Doepfer_Power_16pin, P5 Doepfer_Power_10pin, P6 Doepfer_Power_16pin, P7 Doepfer_Power_10pin, P8 Doepfer_Power_16pin, P9 Doepfer_Power_10pin, T1 Transformer_1P_2S

Commit message: +5V +/-12 sch
Parts:
- removed D1: D_Bridge_+-AA, symbol Device:D_Bridge_+-AA
- removed JP1, JP2, JP3, JP4: Jumper_2_Bridged, symbol Jumper:Jumper_2_Bridged
- removed T1: Transformer_1P_2S, Transformers_SMPS_ThroughHole:ETD29_13Pin_Horizontal_EPCOS-B66359A1013T, symbol Device:Transformer_1P_2S
- added C1, C2, C3, C4, C5, C6: 1000uF, Capacitor_THT:CP_Radial_D8.0mm_P3.80mm, symbol Device:CP
- added C10, C11, C12, C13, C14, C15, C?: 100n, symbol Device:C_Small
- added C7, C8, C9: 1000uF, Capacitor_THT:CP_Radial_D8.0mm_P3.80mm, symbol Device:CP_Small
- added FL1, FL2, FL3: EMI_Filter_CommonMode, Choke_Toroid_ThroughHole:Transformer_Toroid_horizontal_Diameter9mm_Amidon-T30, symbol Device:EMI_Filter_CommonMode
- added J1, J? (x2): Conn_01x03_Male, TerminalBlock:TerminalBlock_Altech_AK300-3_P5.00mm, symbol Connector:Conn_01x03_Male
- added J2, J? (x2): Conn_01x02_Male, TerminalBlock:TerminalBlock_Altech_AK300-2_P5.00mm, symbol Connector:Conn_01x02_Male
- added RV1, RV2: Varistor, Varistor:RV_Disc_D12mm_W4.8mm_P7.5mm, symbol Device:Varistor
- added U1, U2: LM7812_TO220, Package_TO_SOT_THT:TO-220-3_Vertical, symbol Regulator_Linear:LM7812_TO220
- added U3: LM7805_TO220, Package_TO_SOT_THT:TO-220-3_Vertical, symbol Regulator_Linear:LM7805_TO220
- renumbered F3 to F2, F2 to F3, RV1 to RV3
Connections:
- net labels added: +15v-ext, +5V-ext, -15v-ext
- wire segments 360 -> 446

Commit message: Footprint updates
Parts:
- removed C10, C11, C12: 100n, symbol Device:C_Small
- removed P13, P14: Doepfer_Power_10pin, Connectors_IDC:IDC-Header_2x05_Pitch2.54mm_Straight, symbol Eurorack:Doepfer_Power_10pin
- added C1, C16, C17, C18, C19, C2, C20, C21, C22, C23, C24, C25, C26, C27, C28, C29, C30, C31, C32, C33, C34, C35, C36, C37, C38, C39, C40, C41, C42: 100n, Capacitor_SMD:C_0805_2012Metric_Pad1.15x1.40mm_HandSolder, symbol Device:C_Small
- added D1, D2, D6: 1N4001, Diode_THT:D_DO-41_SOD81_P10.16mm_Horizontal, symbol Diode:1N4001
- added D3, D4, D5, D7, D8, D9: LED, LED_SMD:LED_0805_2012Metric_Pad1.15x1.40mm_HandSolder, symbol Device:LED
- added R1, R6: 680R, Resistor_SMD:R_0805_2012Metric_Pad1.15x1.40mm_HandSolder, symbol Device:R
- added R2, R3: 3k3, Resistor_SMD:R_0805_2012Metric_Pad1.15x1.40mm_HandSolder, symbol Device:R
- added R4, R5: 1k5, Resistor_SMD:R_0805_2012Metric_Pad1.15x1.40mm_HandSolder, symbol Device:R
- C10: renamed from C4; footprint Capacitor_THT:CP_Radial_D8.0mm_P3.80mm -> Capacitor_THT:CP_Radial_D10.0mm_P5.00mm
- C13, C14, C15: footprint (none) -> Capacitor_SMD:C_0805_2012Metric_Pad1.15x1.40mm_HandSolder
- C3: renamed from C1; footprint Capacitor_THT:CP_Radial_D8.0mm_P3.80mm -> Capacitor_THT:CP_Radial_D10.0mm_P5.00mm
- C8: renamed from C?; footprint (none) -> Capacitor_SMD:C_0805_2012Metric_Pad1.15x1.40mm_HandSolder
- U3: renamed from U2; value LM7812_TO220 -> LM7912_TO220; symbol Regulator_Linear:LM7812_TO220 -> Regulator_Linear:LM7912_TO220
- gave numbers to parts that had none: 4
- renumbered C5 to C11, C6 to C12, C2 to C4, C3 to C5, C7 to C6, C8 to C7, F3 to F2, F2 to F3, FL3 to FL2, FL2 to FL3, J1 to J5, RV3 to RV2, RV2 to RV3, U3 to U2
Connections:
- net labels added: +15v-int, -15v-int, Vin+15, Vin-15, VinGND
- net labels removed: +15v-ext, -15v-ext
- wire segments 446 -> 486

Commit message: Component placement update
Parts:
- added C13, C5: 1000uF, Capacitor_THT:CP_Radial_D10.0mm_P5.00mm, symbol Device:CP
- C10: renamed from C9; footprint Capacitor_THT:CP_Radial_D8.0mm_P3.80mm -> Capacitor_THT:CP_Radial_D10.0mm_P5.00mm
- C14: renamed from C12; footprint Capacitor_THT:CP_Radial_D8.0mm_P3.80mm -> Capacitor_THT:CP_Radial_D10.0mm_P5.00mm
- C6: renamed from C5; footprint Capacitor_THT:CP_Radial_D8.0mm_P3.80mm -> Capacitor_THT:CP_Radial_D10.0mm_P5.00mm
- C8: renamed from C7; footprint Capacitor_THT:CP_Radial_D8.0mm_P3.80mm -> Capacitor_THT:CP_Radial_D10.0mm_P5.00mm
- renumbered C10 to C11, C11 to C12, C13 to C15, C14 to C16, C15 to C17, C16 to C18, C17 to C19, C18 to C20, C19 to C21, C20 to C22, C21 to C23, C22 to C24, C23 to C25, C24 to C26, C25 to C27, C26 to C28, C27 to C29, C28 to C30, C29 to C31, C30 to C32, C31 to C33, C32 to C34, C33 to C35, C34 to C36, C35 to C37, C36 to C38, C37 to C39, C38 to C40, C39 to C41, C40 to C42, C41 to C43, C42 to C44, C6 to C7, C8 to C9
Connections:
- wire segments 486 -> 494

Commit message: Virtual GND
Parts:
- added C45, C46: 220n, Capacitor_SMD:C_0805_2012Metric_Pad1.15x1.40mm_HandSolder, symbol Device:C_Small
- added Q1: BD139, Package_TO_SOT_THT:TO-126-3_Vertical, symbol Transistor_BJT:BD139
- added Q2: BD140, Package_TO_SOT_THT:TO-126-3_Vertical, symbol Transistor_BJT:BD140
- added R10, R8, R9: 330r, Resistor_SMD:R_0805_2012Metric_Pad1.15x1.40mm_HandSolder, symbol Device:R
- added R11, R7: 10r, Resistor_THT:R_Axial_DIN0204_L3.6mm_D1.6mm_P2.54mm_Vertical, symbol Device:R
- added TP1, TP2, TP3, TP4: TestPoint, Connector_PinSocket_2.54mm:PinSocket_1x01_P2.54mm_Vertical, symbol Connector:TestPoint
- added U4: TL071, Package_DIP:DIP-8_W7.62mm_Socket, symbol Amplifier_Operational:TL071
Connections:
- wire segments 494 -> 530

Commit message: Fixed missing +12V on several connectors
Parts:
- added JP1, JP2: Jumper_2_Open, Connector_PinSocket_2.54mm:PinSocket_1x02_P2.54mm_Vertical, symbol Jumper:Jumper_2_Open
- TP1, TP3: value TestPoint -> VGnd
- TP2: value TestPoint -> Vin+15
- TP4: value TestPoint -> Vin-15
Connections:
- net labels added: GNDPWR
- wire segments 530 -> 558
Changed lines of the file:
@@
 encoding utf-8
 Sheet 1 1
-Title ""
-Date ""
-Rev ""
-Comp ""
+Title "Eurorack Power"
+Date "2019-01-08"
+Rev "Rev A"
+Comp "Johansen Engineering"
 Comment1 ""
 Comment2 ""
@@
 Connection ~ 2550 4250
 Wire Wire Line
-	1500 4650 1850 4650
+	1500 4650 1700 4650
 Wire Wire Line
 	2550 4950 2550 5100
@@
 	2600 4850 2800 4850
 Wire Wire Line
-	2550 4650 2850 4650
+	2550 4650 2700 4650
 Wire Wire Line
 	2550 4750 2650 4750
@@
 Connection ~ 5050 4250
 Wire Wire Line
-	4000 4650 4350 4650
+	4000 4650 4200 4650
 Wire Wire Line
 	5050 4950 5050 5100
@@
 Wire Wire Line
 	5100 4850 5300 4850
-Wire Wire Line
-	5050 4650 5350 4650
 Wire Wire Line
 	5050 4750 5150 4750
@@
 Connection ~ 2600 5650
 Wire Wire Line
-	1550 6050 1900 6050
+	1550 6050 1750 6050
 Wire Wire Line
 	2600 6350 2600 6500
@@
 	2650 6250 2850 6250
 Wire Wire Line
-	2600 6050 2900 6050
+	2600 6050 2750 6050
 Wire Wire Line
 	2600 6150 2700 6150
@@
 Connection ~ 5100 5650
 Wire Wire Line
-	4050 6050 4400 6050
-Wire Wire Line
 	5100 6350 5100 6500
 Wire Wire Line
@@
 	5150 6250 5350 6250
 Wire Wire Line
-	5100 6050 5400 6050
+	5100 6050 5250 6050
 Wire Wire Line
 	5100 6150 5200 6150
@@
 Connection ~ 1800 1400
 Wire Wire Line
-	1800 1400 2250 1400
-Wire Wire Line
 	1800 1000 1900 1000
 $Comp
@@
 P 7300 2800
 F 0 "TP2" H 7358 2920 50  0000 L CNN
-F 1 "TestPoint" H 7358 2829 50  0000 L CNN
+F 1 "Vin+15" H 7358 2829 50  0000 L CNN
 F 2 "Connector_PinSocket_2.54mm:PinSocket_1x01_P2.54mm_Vertical" H 7500 2800 50  0001 C CNN
 F 3 "~" H 7500 2800 50  0001 C CNN
@@
 P 7300 3800
 F 0 "TP4" H 7242 3827 50  0000 R CNN
-F 1 "TestPoint" H 7242 3918 50  0000 R CNN
+F 1 "Vin-15" H 7242 3918 50  0000 R CNN
 F 2 "Connector_PinSocket_2.54mm:PinSocket_1x01_P2.54mm_Vertical" H 7500 3800 50  0001 C CNN
 F 3 "~" H 7500 3800 50  0001 C CNN
@@
 P 9500 3300
 F 0 "TP3" H 9558 3420 50  0000 L CNN
-F 1 "TestPoint" H 9558 3329 50  0000 L CNN
+F 1 "VGnd" H 9558 3329 50  0000 L CNN
 F 2 "Connector_PinSocket_2.54mm:PinSocket_1x01_P2.54mm_Vertical" H 9700 3300 50  0001 C CNN
 F 3 "~" H 9700 3300 50  0001 C CNN
@@
 P 8400 1350
 F 0 "TP1" H 8458 1470 50  0000 L CNN
-F 1 "TestPoint" H 8458 1379 50  0000 L CNN
+F 1 "VGnd" H 8458 1379 50  0000 L CNN
 F 2 "Connector_PinSocket_2.54mm:PinSocket_1x01_P2.54mm_Vertical" H 8600 1350 50  0001 C CNN
 F 3 "~" H 8600 1350 50  0001 C CNN
@@
 Wire Wire Line
 	9500 3300 10000 3300
+$Comp
+L Jumper:Jumper_2_Open JP1
+U 1 1 5EE86F91
+P 10000 550
+F 0 "JP1" H 10000 785 50  0000 C CNN
+F 1 "Jumper_2_Open" H 10000 694 50  0000 C CNN
+F 2 "Connector_PinSocket_2.54mm:PinSocket_1x02_P2.54mm_Vertical" H 10000 550 50  0001 C CNN
+F 3 "~" H 10000 550 50  0001 C CNN
+	1    10000 550
+	1    0    0    -1
+$EndComp
+$Comp
+L Jumper:Jumper_2_Open JP2
+U 1 1 5EE87089
+P 10000 2250
+F 0 "JP2" H 10000 2485 50  0000 C CNN
+F 1 "Jumper_2_Open" H 10000 2394 50  0000 C CNN
+F 2 "Connector_PinSocket_2.54mm:PinSocket_1x02_P2.54mm_Vertical" H 10000 2250 50  0001 C CNN
+F 3 "~" H 10000 2250 50  0001 C CNN
+	1    10000 2250
+	1    0    0    -1
+$EndComp
+Wire Wire Line
+	9800 2250 9600 2250
+Wire Wire Line
+	9600 2250 9600 1900
+Wire Wire Line
+	10200 2250 10500 2250
+Wire Wire Line
+	10500 2250 10500 1900
+Wire Wire Line
+	9800 550  9600 550
+Wire Wire Line
+	9600 550  9600 800
+Wire Wire Line
+	10200 550  10500 550
+Wire Wire Line
+	10500 550  10500 800
+$Comp
+L power:GNDPWR #PWR0101
+U 1 1 5EFB27D4
+P 1300 1400
+F 0 "#PWR0101" H 1300 1200 50  0001 C CNN
+F 1 "GNDPWR" H 1304 1246 50  0000 C CNN
+F 2 "" H 1300 1350 50  0001 C CNN
+F 3 "" H 1300 1350 50  0001 C CNN
+	1    1300 1400
+	1    0    0    -1
+$EndComp
+$Comp
+L power:PWR_FLAG #FLG0103
+U 1 1 5EFB29F6
+P 1500 1400
+F 0 "#FLG0103" H 1500 1475 50  0001 C CNN
+F 1 "PWR_FLAG" H 1500 1573 50  0000 C CNN
+F 2 "" H 1500 1400 50  0001 C CNN
+F 3 "~" H 1500 1400 50  0001 C CNN
+	1    1500 1400
+	-1   0    0    1
+$EndComp
+Wire Wire Line
+	5050 4650 5200 4650
+Wire Wire Line
+	1800 1400 2250 1400
+Wire Wire Line
+	5200 4650 5200 5250
+Wire Wire Line
+	5200 5250 4200 5250
+Wire Wire Line
+	4200 5250 4200 4650
+Connection ~ 5200 4650
+Wire Wire Line
+	5200 4650 5350 4650
+Connection ~ 4200 4650
+Wire Wire Line
+	4200 4650 4350 4650
+Wire Wire Line
+	5250 6050 5250 6650
+Wire Wire Line
+	5250 6650 4250 6650
+Wire Wire Line
+	4250 6650 4250 6050
+Wire Wire Line
+	4050 6050 4250 6050
+Connection ~ 5250 6050
+Wire Wire Line
+	5250 6050 5400 6050
+Connection ~ 4250 6050
+Wire Wire Line
+	4250 6050 4400 6050
+Wire Wire Line
+	1700 4650 1700 5250
+Wire Wire Line
+	1700 5250 2700 5250
+Wire Wire Line
+	2700 5250 2700 4650
+Connection ~ 1700 4650
+Wire Wire Line
+	1700 4650 1850 4650
+Connection ~ 2700 4650
+Wire Wire Line
+	2700 4650 2850 4650
+Wire Wire Line
+	1750 6050 1750 6650
+Wire Wire Line
+	1750 6650 2750 6650
+Wire Wire Line
+	2750 6650 2750 6050
+Connection ~ 1750 6050
+Wire Wire Line
+	1750 6050 1900 6050
+Connection ~ 2750 6050
+Wire Wire Line
+	2750 6050 2900 6050
 $EndSCHEMATC

Commit message: Added SMD 0R to Virtual GND pwr feed
Parts:
- added R12, R13: 0R, Resistor_SMD:R_0805_2012Metric_Pad1.15x1.40mm_HandSolder, symbol Device:R
Connections:
- wire segments 558 -> 560
Changed lines of the file:
@@
 Wire Wire Line
 	7700 2800 8350 2800
-Text GLabel 6900 3800 0    50   Input ~ 0
+Text GLabel 6550 3800 0    50   Input ~ 0
 Vin-15
-Text GLabel 6900 2800 0    50   Input ~ 0
+Text GLabel 6550 2800 0    50   Input ~ 0
 Vin+15
 Text GLabel 10000 3300 2    50   Input ~ 0
@@
 Wire Wire Line
 	2750 6050 2900 6050
+Wire Wire Line
+	6550 2800 6600 2800
+$Comp
+L Device:R R12
+U 1 1 5F1896F0
+P 6750 2800
+F 0 "R12" V 6543 2800 50  0000 C CNN
+F 1 "0R" V 6634 2800 50  0000 C CNN
+F 2 "Resistor_SMD:R_0805_2012Metric_Pad1.15x1.40mm_HandSolder" V 6680 2800 50  0001 C CNN
+F 3 "~" H 6750 2800 50  0001 C CNN
+	1    6750 2800
+	0    1    1    0
+$EndComp
+$Comp
+L Device:R R13
+U 1 1 5F18996D
+P 6750 3800
+F 0 "R13" V 6543 3800 50  0000 C CNN
+F 1 "0R" V 6634 3800 50  0000 C CNN
+F 2 "Resistor_SMD:R_0805_2012Metric_Pad1.15x1.40mm_HandSolder" V 6680 3800 50  0001 C CNN
+F 3 "~" H 6750 3800 50  0001 C CNN
+	1    6750 3800
+	0    1    1    0
+$EndComp
+Wire Wire Line
+	6600 3800 6550 3800
 $EndSCHEMATC
