File: KicadEuropower.kicad_pcb (KiCad board)
At the start: 2 copper layers, 100 x 100 mm, 109 parts, among them J1 Conn_01x02_Male, J2 Conn_01x02_Male, J3 Conn_01x02_Male, J4 Conn_01x03_Male, J5 Conn_01x03_Male, J6 Conn_01x03_Male, P1 Doepfer_Power_10pin, P10 Doepfer_Power_10pin, P11 Doepfer_Power_10pin, P12 Doepfer_Power_10pin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

Commit message: Gerber
Parts:
- added R12: 0R, Resistor_SMD:R_0805_2012Metric_Pad1.15x1.40mm_HandSolder, B.Cu at (7.50, 22.0)
- added R13: 0R, Resistor_SMD:R_0805_2012Metric_Pad1.15x1.40mm_HandSolder, B.Cu at (10.5, 22.0)
- TP1: value TestPoint -> VGnd
- moved C9 3.77 mm to (85.2, 2.75)
- moved R9 3.25 mm to (2.75, 30.5)
- moved TP2 1.00 mm to (6.00, 29.0)
- moved TP3 0.25 mm to (6.00, 32.8)
Connections:
- C45 pad 1: Vin+15 -> Net-(C45-Pad1)
- C46 pad 2: Vin-15 -> Net-(C46-Pad2)
- P1 pad 10: Net-(P1-Pad10) -> +12V
- P1 pad 9: Net-(P1-Pad10) -> +12V
- P2 pad 9: Net-(P1-Pad10) -> +12V
- P3 pad 10: Net-(P3-Pad10) -> +12V
- P3 pad 9: Net-(P3-Pad10) -> +12V
- P4 pad 9: Net-(P3-Pad10) -> +12V
- P5 pad 10: Net-(P5-Pad10) -> +12V
- P5 pad 9: Net-(P5-Pad10) -> +12V
- P6 pad 9: Net-(P5-Pad10) -> +12V
- P7 pad 10: Net-(P7-Pad10) -> +12V
- P7 pad 9: Net-(P7-Pad10) -> +12V
- P8 pad 9: Net-(P7-Pad10) -> +12V
- R10 pad 2: Vin-15 -> Net-(C46-Pad2)
- R11 pad 2: Vin-15 -> Net-(C46-Pad2)
- R7 pad 2: Vin+15 -> Net-(C45-Pad1)
- R8 pad 1: Vin+15 -> Net-(C45-Pad1)
- TP2 pad 1: Vin+15 -> Net-(C45-Pad1)
- TP4 pad 1: Vin-15 -> Net-(C46-Pad2)
- U4 pad 4: Vin-15 -> Net-(C46-Pad2)
- U4 pad 7: Vin+15 -> Net-(C45-Pad1)
Routing:
- net +5V: track 0.00 -> 331.1 mm, vias 0 -> 4
- net +12V: track 0.00 -> 324.7 mm, vias 0 -> 5
- net -12V: track 0.00 -> 270.9 mm, vias 0 -> 2
- net GND: track 0.00 -> 92.1 mm, vias 0 -> 4
- net CV: track 0.00 -> 71.5 mm
- net Gate: track 0.00 -> 69.1 mm
- net Vin-15: track 0.00 -> 61.5 mm, vias 0 -> 5
- net Vin+15: track 0.00 -> 46.6 mm
- net Net-(C46-Pad2): track 0.00 -> 40.4 mm
- net Net-(C11-Pad2): track 0.00 -> 39.7 mm
- net /+5V-ext: track 0.00 -> 33.7 mm
- net Net-(C3-Pad1): track 0.00 -> 31.0 mm, vias 0 -> 2
- net Net-(C45-Pad1): track 0.00 -> 21.9 mm, vias 0 -> 1
- net Net-(C10-Pad1): track 0.00 -> 21.6 mm
- net VinGND: track 0.00 -> 19.9 mm, vias 0 -> 2
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
Commit message: Minor Update to PCB - New Gerber
Parts:
- moved C23 112.0 mm to (161.2, 122.1)
- moved C7 111.8 mm to (163.5, 60.9)
- moved FL2 111.8 mm to (165.3, 73.0)
- moved P6 111.8 mm to (134.3, 121.0)
- moved C1 111.8 mm to (153.5, 66.5)
- moved C10 111.8 mm to (162.9, 85.0)
- moved C11 111.8 mm to (138.4, 85.0)
- moved C12 111.8 mm to (139.2, 60.9)
- moved C13 111.8 mm to (148.3, 98.3)
- moved C14 111.8 mm to (148.3, 120.5)
- moved C15 111.8 mm to (141.0, 66.5)
- moved C16 111.8 mm to (124.9, 122.1)
- moved C17 111.8 mm to (175.9, 122.4)
- moved C18 111.8 mm to (175.9, 99.5)
- moved C19 111.8 mm to (161.2, 99.5)
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Routing:
- net -12V: track 270.9 -> 302.5 mm, vias 2 -> 3
- net +12V: track 324.7 -> 349.2 mm
- net +5V: track 331.1 -> 339.0 mm, vias 4 -> 2
Other:
- board text added: "+12"
- board text added: "+5"
- board text added: "-12"
- board text added: "CV"
- board text added: "Gate"

Commit message: Optional TO252 regulators and added mounting holes
Parts:
- added REF**: MountingHole_2.2mm_M2_ISO7380, MountingHole:MountingHole_2.2mm_M2_ISO7380, F.Cu at (128.2, 103.4)
- added REF**: MountingHole_2.2mm_M2_ISO7380, MountingHole:MountingHole_2.2mm_M2_ISO7380, F.Cu at (172.2, 103.4)
- added U5: LM78M05_TO252, Package_TO_SOT_SMD:TO-252-3_TabPin2, B.Cu at (166.2, 72.2)
- added U6: LM78M12_TO252, Package_TO_SOT_SMD:TO-252-3_TabPin2, B.Cu at (152.2, 72.2)
- added U7: MC79M12_TO252, Package_TO_SOT_SMD:TO-252-3_TabPin2, B.Cu at (139.8, 72.3)
- moved D1 6.27 mm to (131.5, 81.8)
- moved TP1 6.27 mm to (131.5, 84.8)
- moved D2 0.59 mm to (173.3, 90.5)
Connections:
- net /+15v-int renamed +15V
- net /-15v-int renamed -15V
- net Net-(C2-Pad1) renamed +7.5V
- Q2 pad 1: Net-(Q2-Pad1) -> VinGND
- R11 pad 1: Net-(Q2-Pad1) -> VinGND
Routing:
- net GND: track 92.1 -> 116.9 mm, vias 4 -> 24
- net -15V: track 17.1 -> 40.0 mm, vias 0 -> 8
- net +7.5V: track 16.8 -> 27.8 mm
- net +15V: track 17.0 -> 23.2 mm
- net +5V: track 339.0 -> 344.2 mm
- net Net-(D1-Pad2): track 11.5 -> 15.4 mm
- net +12V: track 349.2 -> 352.5 mm
- net Net-(Q2-Pad1): track 3.12 -> 0.00 mm
- net VinGND: track 19.9 -> 23.1 mm
- net Net-(C3-Pad1): track 31.0 -> 33.2 mm
- net -12V: track 302.5 -> 304.6 mm
- net Net-(C10-Pad1): track 21.6 -> 22.2 mm
Other:
- outline, holes or cut-outs redrawn
- board text added: "Rev B - 2019/03"
- board text removed: "Rev A - 2019/02"
