File: KicadEuropower.sch (KiCad schematic (older format))
At the start: 107 parts, among them J1 Conn_01x02_Male, J2 Conn_01x02_Male, J3 Conn_01x02_Male, J4 Conn_01x03_Male, J5 Conn_01x03_Male, J6 Conn_01x03_Male, P1 Doepfer_Power_10pin, P10 Doepfer_Power_10pin, P11 Doepfer_Power_10pin, P12 Doepfer_Power_10pin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

Commit message: Extra reg
Parts:
- added U5: LM78M05_TO252, Package_TO_SOT_SMD:TO-252-3_TabPin2, symbol Regulator_Linear:LM78M05_TO252
- added U6: LM78M12_TO252, Package_TO_SOT_SMD:TO-252-3_TabPin2, symbol Regulator_Linear:LM78M05_TO252
- added U7: MC79M12_TO252, Package_TO_SOT_SMD:TO-252-3_TabPin2, symbol Regulator_Linear:MC79M12_TO252
Connections:
- net labels added: +15V, +7.5V, -15V
- net labels removed: +15v-int, -15v-int
- wire segments 560 -> 566
Other:
- moved on the sheet: C45, C46, Q1, Q2, R10, R11, R12, R13, R7, R8, R9, TP2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

Commit message: Rev B Gerber
Gerber export
Schematic Update (visual)
Cleanup of Rev A
Other:
- note added: "Modular Power Output"
- note added: "Power and decoupling"
- note added: "Regulation"
- note added: "Virtual GND"
- moved on the sheet: C45, C46, Q1, Q2, R10, R11, R12, R13, R7, R8, R9, TP2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
