File: KicadEuropower.sch (KiCad schematic (older format))
At the start: 112 parts, among them J1 Conn_01x02_Male, J2 Conn_01x02_Male, J3 Conn_01x02_Male, J4 Conn_01x03_Male, J5 Conn_01x03_Male, J6 Conn_01x03_Male, P1 Doepfer_Power_10pin, P10 Doepfer_Power_10pin, P11 Doepfer_Power_10pin, P12 Doepfer_Power_10pin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

Commit message: Diode bridge replacing diodes in +-12v - VGND gets fused pwr - +5V on 1812 fuse
Parts:
- removed D1, D6: 1N4001, Diode_THT:D_DO-41_SOD81_P10.16mm_Horizontal, symbol Diode:1N4001
- removed F2: 750mA, Fuse:Fuseholder_Blade_Mini_Keystone_3568, symbol Device:Fuse_Small
- added C? (x2): 220n, Capacitor_SMD:C_0805_2012Metric_Pad1.15x1.40mm_HandSolder, symbol Device:C_Small
- added D?: B125C800DM - DB107, Diode_THT:Diode_Bridge_DIP-4_W7.62mm_P5.08mm, symbol Diode_Bridge:B125C800DM
- added F?: 750mA, Fuse:Fuse_1812_4532Metric_Pad1.30x3.40mm_HandSolder, symbol Device:Fuse_Small
- C9: value 100n -> 10n
- FL1: footprint Choke_Toroid_ThroughHole:Transformer_Toroid_horizontal_Diameter9mm_Amidon-T30 -> Choke_Toroid_D9mm_T30
- FL3: footprint Choke_Toroid_ThroughHole:Transformer_Toroid_horizontal_Diameter9mm_Amidon-T30 -> Choke_Toroid-D9mm_T30
Connections:
- net +5V-ext: now also F?.1
- net Vin+15: now also F1.2, RV1.1, D?.4 (~~); no longer C3.1, F1.1, FL1.3, J4.1 (Pin_1), J5.1 (Pin_1), R2.1, R3.1
- net Vin-15: now also F3.2, RV3.2, D?.3 (~~); no longer C11.2, D4.1 (K), D5.1 (K), F3.1, FL3.1, J4.3 (Pin_3), J5.3 (Pin_3)
- net VinGND: now also C?.1, C?.2; no longer Q2.1 (E), R11.1
- net at D2.2 (A), RV2.1: now also F?.2
- net at Q1.2 (C), R7.1: now also C?.1
- new net: C?.2, Q2.1 (E), R11.1
- new net: C3.1, D?.1 (+), FL1.3
- new net: C11.2, D?.2 (-), FL3.1
- new net V+15: F1.1, J4.1 (Pin_1), J5.1 (Pin_1), R2.1, R3.1
- new net V-15: D4.1 (K), D5.1 (K), F3.1, J4.3 (Pin_3), J5.3 (Pin_3)
Other:
- moved on the sheet: D4, D5, F1, F3, J4, J5, R2, R3, RV1, RV3, U5, U6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

Commit message: fuses +5V and +-12 changed to 1210
Parts:
- F? (x3): footprint Fuse:Fuse_1812_4532Metric_Pad1.30x3.40mm_HandSolder -> Fuse:Fuse_1210_3225Metric_Pad1.42x2.65mm_HandSolder
Changed lines of the file:
@@
 F 0 "F?" H 10400 2135 50  0000 C CNN
 F 1 "750mA" H 10400 2044 50  0000 C CNN
-F 2 "Fuse:Fuse_1812_4532Metric_Pad1.30x3.40mm_HandSolder" H 10400 1950 50  0001 C CNN
+F 2 "Fuse:Fuse_1210_3225Metric_Pad1.42x2.65mm_HandSolder" H 10400 1950 50  0001 C CNN
 F 3 "~" H 10400 1950 50  0001 C CNN
 	1    10400 1950
@@
 F 0 "F?" H 10400 1035 50  0000 C CNN
 F 1 "750mA" H 10400 944 50  0000 C CNN
-F 2 "Fuse:Fuse_1812_4532Metric_Pad1.30x3.40mm_HandSolder" H 10400 850 50  0001 C CNN
+F 2 "Fuse:Fuse_1210_3225Metric_Pad1.42x2.65mm_HandSolder" H 10400 850 50  0001 C CNN
 F 3 "~" H 10400 850 50  0001 C CNN
 	1    10400 850
@@
 F 0 "F?" H 1650 1185 50  0000 C CNN
 F 1 "750mA" H 1650 1094 50  0000 C CNN
-F 2 "Fuse:Fuse_1812_4532Metric_Pad1.30x3.40mm_HandSolder" H 1650 1000 50  0001 C CNN
+F 2 "Fuse:Fuse_1210_3225Metric_Pad1.42x2.65mm_HandSolder" H 1650 1000 50  0001 C CNN
 F 3 "~" H 1650 1000 50  0001 C CNN
 	1    1650 1000

Commit message: SCH fixed VGND err
Parts:
- R10, R8: value 330r -> 3k30
Connections:
- net VinGND: now also Q2.1 (E); no longer Q2.2 (C)
- net at C?.2, R11.1: now also Q2.2 (C); no longer Q2.1 (E)
Changed lines of the file:
@@
 P 7900 5150
 F 0 "R8" H 7970 5196 50  0000 L CNN
-F 1 "330r" H 7970 5105 50  0000 L CNN
+F 1 "3k30" H 7970 5105 50  0000 L CNN
 F 2 "Resistor_SMD:R_0805_2012Metric_Pad1.15x1.40mm_HandSolder" V 7830 5150 50  0001 C CNN
 F 3 "~" H 7900 5150 50  0001 C CNN
@@
 P 7900 5550
 F 0 "R10" H 7970 5596 50  0000 L CNN
-F 1 "330r" H 7970 5505 50  0000 L CNN
+F 1 "3k30" H 7970 5505 50  0000 L CNN
 F 2 "Resistor_SMD:R_0805_2012Metric_Pad1.15x1.40mm_HandSolder" V 7830 5550 50  0001 C CNN
 F 3 "~" H 7900 5550 50  0001 C CNN
@@
 F 3 "http://www.st.com/internet/com/TECHNICAL_RESOURCES/TECHNICAL_LITERATURE/DATASHEET/CD00001225.pdf" H 9600 5650 50  0001 L CNN
 	1    9600 5650
-	1    0    0    -1
+	1    0    0    1
 $EndComp
 Wire Wire Line
@@
 Wire Wire Line
 	10100 5450 9925 5450
-Connection ~ 9700 5450
 Wire Wire Line
 	8300 5750 8300 5950
@@
 	1    0    0    -1
 $EndComp
+Connection ~ 9700 5450
 $EndSCHEMATC

Commit message: Measurements
Parts:
- R1: value 680R -> 4k7
- R10, R8: value 3k30 -> 4k70
- R2, R3: value 3k3 -> 10k
- R4, R5: value 3k3 -> 4k7
Changed lines of the file:
@@
 P 750 1150
 F 0 "J1" H 856 1328 50  0000 C CNN
-F 1 "Conn_01x02_Male" H 856 1237 50  0000 C CNN
+F 1 "Conn_01x02_Male" H 750 1125 50  0000 C CNN
 F 2 "TerminalBlock:TerminalBlock_Altech_AK300-2_P5.00mm" H 750 1150 50  0001 C CNN
 F 3 "~" H 750 1150 50  0001 C CNN
@@
 P 4600 2375
 F 0 "R4" V 4393 2375 50  0000 C CNN
-F 1 "3k3" V 4484 2375 50  0000 C CNN
+F 1 "4k7" V 4484 2375 50  0000 C CNN
 F 2 "Resistor_SMD:R_0805_2012Metric_Pad1.15x1.40mm_HandSolder" V 4530 2375 50  0001 C CNN
 F 3 "~" H 4600 2375 50  0001 C CNN
@@
 P 4900 1975
 F 0 "R5" V 5107 1975 50  0000 C CNN
-F 1 "3k3" V 5016 1975 50  0000 C CNN
+F 1 "4k7" V 5016 1975 50  0000 C CNN
 F 2 "Resistor_SMD:R_0805_2012Metric_Pad1.15x1.40mm_HandSolder" V 4830 1975 50  0001 C CNN
 F 3 "~" H 4900 1975 50  0001 C CNN
@@
 P 650 1000
 F 0 "R1" H 720 1046 50  0000 L CNN
-F 1 "680R" H 720 955 50  0000 L CNN
+F 1 "4k7" H 720 955 50  0000 L CNN
 F 2 "Resistor_SMD:R_0805_2012Metric_Pad1.15x1.40mm_HandSolder" V 580 1000 50  0001 C CNN
 F 3 "~" H 650 1000 50  0001 C CNN
@@
 P 7000 2950
 F 0 "R3" H 7070 2996 50  0000 L CNN
-F 1 "3k3" H 7070 2905 50  0000 L CNN
+F 1 "10k" H 7070 2905 50  0000 L CNN
 F 2 "Resistor_SMD:R_0805_2012Metric_Pad1.15x1.40mm_HandSolder" V 6930 2950 50  0001 C CNN
 F 3 "~" H 7000 2950 50  0001 C CNN
@@
 P 6600 2950
 F 0 "R2" H 6670 2996 50  0000 L CNN
-F 1 "3k3" H 6670 2905 50  0000 L CNN
+F 1 "10k" H 6670 2905 50  0000 L CNN
 F 2 "Resistor_SMD:R_0805_2012Metric_Pad1.15x1.40mm_HandSolder" V 6530 2950 50  0001 C CNN
 F 3 "~" H 6600 2950 50  0001 C CNN
@@
 P 7900 5150
 F 0 "R8" H 7970 5196 50  0000 L CNN
-F 1 "3k30" H 7970 5105 50  0000 L CNN
+F 1 "4k70" H 7970 5105 50  0000 L CNN
 F 2 "Resistor_SMD:R_0805_2012Metric_Pad1.15x1.40mm_HandSolder" V 7830 5150 50  0001 C CNN
 F 3 "~" H 7900 5150 50  0001 C CNN
@@
 P 7900 5550
 F 0 "R10" H 7970 5596 50  0000 L CNN
-F 1 "3k30" H 7970 5505 50  0000 L CNN
+F 1 "4k70" H 7970 5505 50  0000 L CNN
 F 2 "Resistor_SMD:R_0805_2012Metric_Pad1.15x1.40mm_HandSolder" V 7830 5550 50  0001 C CNN
 F 3 "~" H 7900 5550 50  0001 C CNN

Commit message: sch
Parts:
- R6: value 1k5 -> 2k2
Changed lines of the file:
@@
 P 3550 2950
 F 0 "R6" V 3343 2950 50  0000 C CNN
-F 1 "1k5" V 3434 2950 50  0000 C CNN
+F 1 "2k2" V 3434 2950 50  0000 C CNN
 F 2 "Resistor_SMD:R_0805_2012Metric_Pad1.15x1.40mm_HandSolder" V 3480 2950 50  0001 C CNN
 F 3 "~" H 3550 2950 50  0001 C CNN
