File: _saved_KicadEuropower.sch (KiCad schematic (older format))
At the start: 113 parts, among them J1 Conn_01x02_Male, J2 Conn_01x02_Male, J3 Conn_01x02_Male, J4 Conn_01x03_Male, J5 Conn_01x03_Male, J6 Conn_01x03_Male, P1 Doepfer_Power_10pin, P10 Doepfer_Power_10pin, P11 Doepfer_Power_10pin, P12 Doepfer_Power_10pin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

Commit message: Measurements
Parts:
- R1: value 680R -> 4k7
- R10, R8: value 3k30 -> 4k70
- R2, R3: value 3k3 -> 10k
- R4, R5: value 3k3 -> 4k7
- R6: value 1k5 -> 2k2
Changed lines of the file:
@@
 P 750 1150
 F 0 "J1" H 856 1328 50  0000 C CNN
-F 1 "Conn_01x02_Male" H 856 1237 50  0000 C CNN
+F 1 "Conn_01x02_Male" H 750 1125 50  0000 C CNN
 F 2 "TerminalBlock:TerminalBlock_Altech_AK300-2_P5.00mm" H 750 1150 50  0001 C CNN
 F 3 "~" H 750 1150 50  0001 C CNN
@@
 P 4600 2375
 F 0 "R4" V 4393 2375 50  0000 C CNN
-F 1 "3k3" V 4484 2375 50  0000 C CNN
+F 1 "4k7" V 4484 2375 50  0000 C CNN
 F 2 "Resistor_SMD:R_0805_2012Metric_Pad1.15x1.40mm_HandSolder" V 4530 2375 50  0001 C CNN
 F 3 "~" H 4600 2375 50  0001 C CNN
@@
 P 4900 1975
 F 0 "R5" V 5107 1975 50  0000 C CNN
-F 1 "3k3" V 5016 1975 50  0000 C CNN
+F 1 "4k7" V 5016 1975 50  0000 C CNN
 F 2 "Resistor_SMD:R_0805_2012Metric_Pad1.15x1.40mm_HandSolder" V 4830 1975 50  0001 C CNN
 F 3 "~" H 4900 1975 50  0001 C CNN
@@
 P 3550 2950
 F 0 "R6" V 3343 2950 50  0000 C CNN
-F 1 "1k5" V 3434 2950 50  0000 C CNN
+F 1 "2k2" V 3434 2950 50  0000 C CNN
 F 2 "Resistor_SMD:R_0805_2012Metric_Pad1.15x1.40mm_HandSolder" V 3480 2950 50  0001 C CNN
 F 3 "~" H 3550 2950 50  0001 C CNN
@@
 P 650 1000
 F 0 "R1" H 720 1046 50  0000 L CNN
-F 1 "680R" H 720 955 50  0000 L CNN
+F 1 "4k7" H 720 955 50  0000 L CNN
 F 2 "Resistor_SMD:R_0805_2012Metric_Pad1.15x1.40mm_HandSolder" V 580 1000 50  0001 C CNN
 F 3 "~" H 650 1000 50  0001 C CNN
@@
 P 7000 2950
 F 0 "R3" H 7070 2996 50  0000 L CNN
-F 1 "3k3" H 7070 2905 50  0000 L CNN
+F 1 "10k" H 7070 2905 50  0000 L CNN
 F 2 "Resistor_SMD:R_0805_2012Metric_Pad1.15x1.40mm_HandSolder" V 6930 2950 50  0001 C CNN
 F 3 "~" H 7000 2950 50  0001 C CNN
@@
 P 6600 2950
 F 0 "R2" H 6670 2996 50  0000 L CNN
-F 1 "3k3" H 6670 2905 50  0000 L CNN
+F 1 "10k" H 6670 2905 50  0000 L CNN
 F 2 "Resistor_SMD:R_0805_2012Metric_Pad1.15x1.40mm_HandSolder" V 6530 2950 50  0001 C CNN
 F 3 "~" H 6600 2950 50  0001 C CNN
@@
 P 7900 5150
 F 0 "R8" H 7970 5196 50  0000 L CNN
-F 1 "3k30" H 7970 5105 50  0000 L CNN
+F 1 "4k70" H 7970 5105 50  0000 L CNN
 F 2 "Resistor_SMD:R_0805_2012Metric_Pad1.15x1.40mm_HandSolder" V 7830 5150 50  0001 C CNN
 F 3 "~" H 7900 5150 50  0001 C CNN
@@
 P 7900 5550
 F 0 "R10" H 7970 5596 50  0000 L CNN
-F 1 "3k30" H 7970 5505 50  0000 L CNN
+F 1 "4k70" H 7970 5505 50  0000 L CNN
 F 2 "Resistor_SMD:R_0805_2012Metric_Pad1.15x1.40mm_HandSolder" V 7830 5550 50  0001 C CNN
 F 3 "~" H 7900 5550 50  0001 C CNN
