File: RevB/KicadEuropower.sch (KiCad schematic (older format))
At the start: 112 parts, among them J1 Conn_01x02_Male, J2 Conn_01x02_Male, J3 Conn_01x02_Male, J4 Conn_01x03_Male, J5 Conn_01x03_Male, J6 Conn_01x03_Male, P1 Doepfer_Power_10pin, P10 Doepfer_Power_10pin, P11 Doepfer_Power_10pin, P12 Doepfer_Power_10pin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

Commit message: Rev C prepare
Parts:
- removed D? (x2): 1N4001, Diode_SMD:D_SOD-123, symbol Diode:1N4001
- removed F? (x2): 750mA, Fuse:Fuse_1812_4532Metric_Pad1.30x3.40mm_HandSolder, symbol Device:Fuse_Small
- added JP1, JP2: Jumper_2_Open, Connector_PinSocket_2.54mm:PinSocket_1x02_P2.54mm_Vertical, symbol Jumper:Jumper_2_Open
- F1, F2, F3: value 750mA -> Fuse_Small
- R4, R5: value 3k3 -> 1k5
- R6: value 1k5 -> 680R
Other:
- moved on the sheet: FL1, FL3, U1, U3
